File: bigboard/bigboard.kicad_pcb (KiCad board)
At the start: 2 copper layers, 99.1 x 48.3 mm, 69 parts, among them J1 motorA, J2 motorB, J3 USB_B_Mini, J4 device2, J5 device1, J6 battery, Q1 BC547, Q2 BC547, Q3 BC547, Q4 BC547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

Commit message: minor stylistic suggestions & path fixes
Parts:
- removed REF** (x4): M3, MountingHole:MountingHole_3.2mm_M3
- removed REF** (x2): M2.5, MountingHole:MountingHole_2.7mm_M2.5
- added H1: MountingHole, MountingHole:MountingHole_3.2mm_M3_DIN965_Pad, F.Cu at (211.0, 123.0)
- added H2: MountingHole, MountingHole:MountingHole_3.2mm_M3_DIN965_Pad, F.Cu at (119.0, 123.0)
- added H3: MountingHole, MountingHole:MountingHole_3.2mm_M3_DIN965_Pad, F.Cu at (119.0, 82.0)
- added H4: MountingHole, MountingHole:MountingHole_3.2mm_M3_DIN965_Pad, F.Cu at (211.0, 82.0)
Connections:
- net A01 renamed Net-(J1-Pad1)
- net A02 renamed Net-(J1-Pad2)
- net B01 renamed Net-(J2-Pad1)
- net BO2 renamed Net-(J2-Pad2)
- net lx renamed Net-(D1-Pad2)
Routing:
- net GND: vias 31 -> 29
- net (no net): vias 0 -> 2
