File: bigboard/bigboard.sch (KiCad schematic (older format))
At the start: 63 parts, among them J1 motorA, J2 motorB, J3 USB_B_Mini, J4 device2, J5 device1, J6 battery, Q1 BC547, Q2 BC547, Q3 BC547, Q4 BC547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

Commit message: minor stylistic suggestions & path fixes
Parts:
- added H1, H2, H3, H4: MountingHole, MountingHole:MountingHole_3.2mm_M3_DIN965_Pad, symbol Mechanical:MountingHole
- J3: symbol Connector:USB_B_Mini -> bigboard-rescue:USB_B_Mini-Connector
- U3: symbol Driver_Motor:TB6612FNG -> bigboard-rescue:TB6612FNG-Driver_Motor
- U4: symbol Interface_USB:FT232RL -> bigboard-rescue:FT232RL-Interface_USB
Connections:
- net labels removed: A01, A02, B01, BO2, ESPen, bat, lx
- wire segments 186 -> 194
Other:
- note added: "Testpoints & Mounting\n"
- note removed: "pin saving inverters"
- note removed: "testpoints\n"
- moved on the sheet: C1, C2, C3, C5, C6, C7, D1, D2, D3, J1, J2, J6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
